Commit message: changed description urdfs

File: src/roseybot_control/description/robot/roseybot_colors.urdf.xacro (robot description, xacro)
@@ -30,5 +30,5 @@
   </material>
   <material name="pink">
-    <color rgba= "${255/192} ${192/255} ${203/255} 1.0"/>
+    <color rgba= "${255/255} ${182/255} ${193/255} 1.0"/>
   </material>
 </robot>

File: src/roseybot_control/description/robot/roseybot_description.urdf.xacro (robot description, xacro)
@@ -3,45 +3,79 @@
 <robot xmlns:xacro="http://www.ros.org/wiki/xacro">
     <!-- properties for robot dimensions (in m)-->
-    <xacro:property name="base_width" value="0.3"/>
-    <xacro:property name="base_length" value="0.3"/>
-    <xacro:property name="base_height" value="0.3"/>
-    <xacro:property name="wheel_radius" value="0.15"/>
+    <xacro:property name="base_width" value="0.422"/>
+    <xacro:property name="base_length" value="0.703"/>
+    <xacro:property name="base_height" value="0.15"/>
+    <xacro:property name="wheel_radius" value="0.1515"/>
     <xacro:property name="wheel_length" value="0.1"/>
-    <xacro:property name="ride_height" value="0.1"/>
+    <xacro:property name="z_offset" value="0.05"/>
+    <xacro:property name="x_offset" value="0.05"/>
+    <xacro:property name="base_mass" value="12"/>
+    <xacro:property name="wheel_mass" value="0.5"/>
+    <!-- Define inertial property macros  -->
+    <xacro:macro name="box_inertia" params="m w h d">
+        <inertial>
+        <origin xyz="0 0 0" rpy="${pi/2} 0 ${pi/2}"/>
+        <mass value="${m}"/>
+        <inertia ixx="${(m/12) * (h*h + d*d)}" ixy="0.0" ixz="0.0" iyy="${(m/12) * (w*w + d*d)}" iyz="0.0" izz="${(m/12) * (w*w + h*h)}"/>
+        </inertial>
+    </xacro:macro>
+    <xacro:macro name="cylinder_inertia" params="m r h">
+        <inertial>
+        <origin xyz="0 0 0" rpy="${pi/2} 0 0" />
+        <mass value="${m}"/>
+        <inertia ixx="${(m/12) * (3*r*r + h*h)}" ixy = "0" ixz = "0" iyy="${(m/12) * (3*r*r + h*h)}" iyz = "0" izz="${(m/2) * (r*r)}"/>
+        </inertial>
+    </xacro:macro>
+    <!-- define base link for rover (Primary Parent Link)-->
     <link name="base_link">
         <collision>
             <origin xyz="0 0 0" rpy= "0 0 0"/>
             <geometry>
-                <box size="${base_width} ${base_length} ${base_height}"/>
+                <box size="${base_length} ${base_width} ${base_height}"/>
             </geometry>
         </collision>
         <visual>
-            <origin xyz="0 0 ${base_height/2}" rpy="0 0 0"/>
+            <origin xyz="0 0 0" rpy="0 0 0"/>
             <geometry>
-                <box size = "${base_width} ${base_length} ${base_height}"/>
+                <box size = "${base_length} ${base_width} ${base_height}"/>
             </geometry>
             <material name="pink"/>
         </visual>
+        <xacro:box_intertia m ="${base_mass}" w="${base_width}" l="${base_length}" h="${base_height}"/>
     </link>
-    <joint name="left_front_wheel_joint" type="continuous">
+    <!-- define footprint of rover-->
+    <link name="base_footprint"/>
+    <joint name="base_joint" type="fixed">
         <parent link="base_link"/>
-        <child link="left_front_wheel_link"/>
-        <origin xyz="${base_length/2} ${base_width} ${ride_height}" rpy= "0 0 0"/>
-        <axis xyz = "0 1 0"/>
+        <child link="base_footprint"/>
+        <origin xyz="0 0 ${- (z_offset + wheel_radius) }"/>
     </joint>
-    <link name="left_front_wheel_link">
-        <collision>
-            <origin xyz="0 0 0" rpy= "0 0 0"/>
-            <geometry>
-                <box size="${base_width} ${base_length} ${base_height}"/>
-            </geometry>
-        </collision>
-        <visual>
-            <origin xyz="0 0 ${base_height/2}" rpy="0 0 0"/>
-            <geometry>
-                <box size = "${base_width} ${base_length} ${base_height}"/>
-            </geometry>
-            <material name="black"/>
-        </visual>
-    </link>
+    <xacro:macro name="wheel" params="prefix x_reflect y_reflect">
+        <joint name="${prefix}_wheel_joint" type="continuous">
+            <parent link="base_link"/>
+            <child link="${prefix}_wheel_link"/>
+            <origin xyz="${x_reflect * ((base_length/2) - x_offset)} ${y_reflect * base_width/2} ${-z_offset}" rpy= "0 0 0"/>
+            <axis xyz = "0 1 0"/>
+        </joint>
+        <link name="${prefix}_wheel_link">
+            <collision>
+                <origin xyz="0 ${wheel_length/2} 0" rpy= "${pi/2} 0 0"/>
+                <geometry>
+                    <cylinder radius="${wheel_radius}" length="${wheel_length}"/>
+                </geometry>
+            </collision>
+            <visual>
+                <origin xyz="0 ${y_reflect * wheel_length/2} 0" rpy="${pi/2} 0 0"/>
+                <geometry>
+                    <cylinder radius="${wheel_radius}" length="${wheel_length}"/>
+                </geometry>
+                <material name="black"/>
+            </visual>
+            <xacro:cylinder_inertia m="${wheel_mass}" r="${wheel_radius}" h="{wheel_length}"/>
+        </link>
+    </xacro:macro>
+    <xacro:wheel prefix="front_left" x_reflect="1" y_reflect="1"/>
+    <xacro:wheel prefix="front_right" x_reflect="1" y_reflect="-1"/>
+    <xacro:wheel prefix="back_left" x_reflect="-1" y_reflect="1"/>
+    <xacro:wheel prefix="back_right" x_reflect="-1" y_reflect="-1"/>
 </robot>

File: src/roseybot_control/description/urdf/roseybot.urdf.xacro (robot description, xacro)
@@ -3,7 +3,7 @@
 <robot xmlns:xacro="http://www.ros.org/wiki/xacro" name="roseybot">
   <xacro:arg name="use_mock_hardware" default="false" />
-  <xacro:include filename="$(find roseybot_control)/description/robot/roseybot_description.urdf.xacro"/>
   <!-- Import Rviz colors -->
   <xacro:include filename="$(find roseybot_control)/description/robot/roseybot_colors.urdf.xacro" />
+    <xacro:include filename="$(find roseybot_control)/description/robot/roseybot_description.urdf.xacro"/>
   <!-- Import diffbot ros2_control description -->
   <!-- <xacro:include filename="$(find ros2_control_demo_example_2)/ros2_control/diffbot.ros2_control.xacro" /> -->
