Commit message: changes to control package

File: src/roseybot_control/description/robot/roseybot_description.urdf.xacro (robot description, xacro)
@@ -26,5 +26,5 @@
     <joint name="left_front_wheel_joint" type="continuous">
         <parent link="base_link"/>
-        <child link="left_front_wheel_joint"/>
+        <child link="left_front_wheel_link"/>
         <origin xyz="${base_length/2} ${base_width} ${ride_height}" rpy= "0 0 0"/>
         <axis xyz = "0 1 0"/>
@@ -42,5 +42,5 @@
                 <box size = "${base_width} ${base_length} ${base_height}"/>
             </geometry>
-            <material name="pink"/>
+            <material name="black"/>
         </visual>
     </link>

Commit message: 2 state interfaces and added ros_control urdf

File: src/roseybot_control/description/robot/roseybot_description.urdf.xacro (robot description, xacro)
@@ -42,5 +42,5 @@
             <material name="pink"/>
         </visual>
-        <xacro:box_intertia m ="${base_mass}" w="${base_width}" l="${base_length}" h="${base_height}"/>
+        <xacro:box_inertia m ="${base_mass}" w="${base_width}" d="${base_length}" h="${base_height}"/>
     </link>
     <!-- define footprint of rover-->
@@ -51,4 +51,5 @@
         <origin xyz="0 0 ${- (z_offset + wheel_radius) }"/>
     </joint>
+    <!-- set up macro for wheel definitions -->
     <xacro:macro name="wheel" params="prefix x_reflect y_reflect">
         <joint name="${prefix}_wheel_joint" type="continuous">
@@ -72,7 +73,8 @@
                 <material name="black"/>
             </visual>
-            <xacro:cylinder_inertia m="${wheel_mass}" r="${wheel_radius}" h="{wheel_length}"/>
+            <xacro:cylinder_inertia m="${wheel_mass}" r="${wheel_radius}" h="${wheel_length}"/>
         </link>
     </xacro:macro>
+    <!-- call macros to define wheels-->
     <xacro:wheel prefix="front_left" x_reflect="1" y_reflect="1"/>
     <xacro:wheel prefix="front_right" x_reflect="1" y_reflect="-1"/>

File: src/roseybot_control/description/ros2_control/roseybot_control.urdf.xacro (robot description, xacro)
@@ -1,6 +1,23 @@
-<!-- <?xml version="1.0"?>
+<?xml version="1.0"?>
 <robot xmlns:xacro="http://www.ros.org/wiki/xacro">
+    <xacro:macro name="connect_joint" params="prefix">
+        <joint name="${prefix}_wheel_joint">
+            <command_interface name="velocity"/>
+            <state_interface name="position"/>
+            <state_interface name="velocity"/>
+            <!-- <state_interface name="current"/>
+            <state_interface name="voltage"/> -->
+      </joint>
+    </xacro:macro>
     <ros2_control name="roseybot_teensy" type="system">
-        <plugin></plugin>
+        <hardware>
+          <plugin>ros2_control_demo_example_2/DiffBotSystemHardware</plugin>
+          <param name="example_param_hw_start_duration_sec">0</param>
+          <param name="example_param_hw_stop_duration_sec">3.0</param>
+        </hardware>
+        <xacro:connect_joint prefix="front_left"/>
+        <xacro:connect_joint prefix="front_right"/>
+        <xacro:connect_joint prefix="back_left"/>
+        <xacro:connect_joint prefix="back_right"/>
     </ros2_control>
-</robot> -->
+</robot>

File: src/roseybot_control/description/urdf/roseybot.urdf.xacro (robot description, xacro)
@@ -7,5 +7,5 @@
     <xacro:include filename="$(find roseybot_control)/description/robot/roseybot_description.urdf.xacro"/>
   <!-- Import diffbot ros2_control description -->
-  <!-- <xacro:include filename="$(find ros2_control_demo_example_2)/ros2_control/diffbot.ros2_control.xacro" /> -->
+  <xacro:include filename="$(find roseybot_control)/description/ros2_control/roseybot_control.urdf.xacro" />
   <!-- <xacro:roseybot prefix="$(arg prefix)" /> -->
   <!-- <xacro:diffbot_ros2_control

Commit message: integrating sim with rosey

File: src/roseybot_control/description/robot/roseybot_description.urdf.xacro (robot description, xacro)
@@ -6,4 +6,5 @@
     <xacro:property name="base_length" value="0.703"/>
     <xacro:property name="base_height" value="0.15"/>
+    <xacro:property name="wheel_track" value="0.315"/>  <!-- center-to-center wheel separation, must match roseybot_controllers.yaml wheel_separation -->
     <xacro:property name="wheel_radius" value="0.1515"/>
     <xacro:property name="wheel_length" value="0.1"/>
@@ -56,5 +57,5 @@
             <parent link="base_link"/>
             <child link="${prefix}_wheel_link"/>
-            <origin xyz="${x_reflect * ((base_length/2) - x_offset)} ${y_reflect * base_width/2} ${-z_offset}" rpy= "0 0 0"/>
+            <origin xyz="${x_reflect * ((base_length/2) - x_offset)} ${y_reflect * wheel_track/2} ${-z_offset}" rpy= "0 0 0"/>
             <axis xyz = "0 1 0"/>
         </joint>
