Commit message: updated motion model wheel radius and separation

File: src/roseybot_control/description/robot/roseybot_description.urdf.xacro (robot description, xacro)
@@ -6,6 +6,6 @@
     <xacro:property name="base_length" value="0.703"/>
     <xacro:property name="base_height" value="0.15"/>
-    <xacro:property name="wheel_track" value="0.315"/>  <!-- center-to-center wheel separation, must match roseybot_controllers.yaml wheel_separation -->
-    <xacro:property name="wheel_radius" value="0.1515"/>
+    <xacro:property name="wheel_track" value="0.3365"/>  <!-- center-to-center wheel separation, must match roseybot_controllers.yaml wheel_separation -->
+    <xacro:property name="wheel_radius" value="0.158"/>
     <xacro:property name="wheel_length" value="0.1"/>
     <xacro:property name="z_offset" value="0.05"/>
