Commit message: some tuning mostly urdf changes

File: src/myrosey_description/urdf/description/roseybot_description.urdf.xacro (robot description, xacro)
@@ -61,5 +61,5 @@
         <link name="${prefix}_wheel_link">
             <collision>
-                <origin xyz="0 ${wheel_length/2} 0" rpy= "${pi/2} 0 0"/>
+                <origin xyz="0 ${y_reflect * wheel_length/2} 0" rpy= "${pi/2} 0 0"/>
                 <geometry>
                     <cylinder radius="${wheel_radius}" length="${wheel_length}"/>

File: src/roseybot_control/description/urdf/roseybot_sim.urdf.xacro (robot description, xacro)
@@ -61,20 +61,20 @@
     <gazebo reference="front_left_wheel_link">
         <collision><surface><friction><ode>
-            <mu>1.2</mu><mu2>0.4</mu2>
+            <mu>1.2</mu><mu2>0.01</mu2>
         </ode></friction></surface></collision>
     </gazebo>
     <gazebo reference="front_right_wheel_link">
         <collision><surface><friction><ode>
-            <mu>1.2</mu><mu2>0.4</mu2>
+            <mu>1.2</mu><mu2>0.01</mu2>
         </ode></friction></surface></collision>
     </gazebo>
     <gazebo reference="back_left_wheel_link">
         <collision><surface><friction><ode>
-            <mu>1.2</mu><mu2>0.4</mu2>
+            <mu>1.2</mu><mu2>0.01</mu2>
         </ode></friction></surface></collision>
     </gazebo>
     <gazebo reference="back_right_wheel_link">
         <collision><surface><friction><ode>
-            <mu>1.2</mu><mu2>0.4</mu2>
+            <mu>1.2</mu><mu2>0.01</mu2>
         </ode></friction></surface></collision>
     </gazebo>
