Commit message: description file now has urdf

File: src/rosey_description/description/robot/roseybot_description.urdf.xacro (robot description, xacro)
@@ -1,83 +1,683 @@
 <?xml version="1.0"?>
-<!-- RoseyBot Robot Description File -->
+<!-- RoseyBot Robot Description File
+     Links, joints, and mass properties come from the SolidWorks to URDF
+     exporter (URDF2 export). Frames follow REP-103/REP-105:
+       - base_footprint is the root, on the ground plane below base_link.
+       - base_footprint, imu_link, and camera_*_optical_link are virtual
+         frames with no mass, inertia, or geometry.
+       - All wheel joints rotate about +y, so a positive velocity drives the
+         robot forward on both sides. -->
 <robot xmlns:xacro="http://www.ros.org/wiki/xacro">
-    <!-- properties for robot dimensions (in m)-->
-    <xacro:property name="base_width" value="0.422"/>
-    <xacro:property name="base_length" value="0.703"/>
-    <xacro:property name="base_height" value="0.15"/>
-    <xacro:property name="wheel_radius" value="0.1515"/>
-    <xacro:property name="wheel_length" value="0.1"/>
-    <xacro:property name="z_offset" value="0.05"/>
-    <xacro:property name="x_offset" value="0.05"/>
-    <xacro:property name="base_mass" value="12"/>
-    <xacro:property name="wheel_mass" value="0.5"/>
-    <!-- Define inertial property macros  -->
-    <xacro:macro name="box_inertia" params="m w h d">
-        <inertial>
-        <origin xyz="0 0 0" rpy="${pi/2} 0 ${pi/2}"/>
-        <mass value="${m}"/>
-        <inertia ixx="${(m/12) * (h*h + d*d)}" ixy="0.0" ixz="0.0" iyy="${(m/12) * (w*w + d*d)}" iyz="0.0" izz="${(m/12) * (w*w + h*h)}"/>
-        </inertial>
-    </xacro:macro>
-    <xacro:macro name="cylinder_inertia" params="m r h">
-        <inertial>
-        <origin xyz="0 0 0" rpy="${pi/2} 0 0" />
-        <mass value="${m}"/>
-        <inertia ixx="${(m/12) * (3*r*r + h*h)}" ixy = "0" ixz = "0" iyy="${(m/12) * (3*r*r + h*h)}" iyz = "0" izz="${(m/2) * (r*r)}"/>
-        </inertial>
-    </xacro:macro>
-    <!-- define base link for rover (Primary Parent Link)-->
-    <link name="base_link">
-        <collision>
-            <origin xyz="0 0 0" rpy= "0 0 0"/>
-            <geometry>
-                <box size="${base_length} ${base_width} ${base_height}"/>
-            </geometry>
-        </collision>
-        <visual>
-            <origin xyz="0 0 0" rpy="0 0 0"/>
-            <geometry>
-                <box size = "${base_length} ${base_width} ${base_height}"/>
-            </geometry>
-            <material name="pink"/>
-        </visual>
-        <xacro:box_inertia m ="${base_mass}" w="${base_width}" d="${base_length}" h="${base_height}"/>
-    </link>
-    <!-- define footprint of rover-->
-    <link name="base_footprint"/>
-    <joint name="base_joint" type="fixed">
-        <parent link="base_link"/>
-        <child link="base_footprint"/>
-        <origin xyz="0 0 ${- (z_offset + wheel_radius) }"/>
-    </joint>
-    <!-- set up macro for wheel definitions -->
-    <xacro:macro name="wheel" params="prefix x_reflect y_reflect">
-        <joint name="${prefix}_wheel_joint" type="continuous">
-            <parent link="base_link"/>
-            <child link="${prefix}_wheel_link"/>
-            <origin xyz="${x_reflect * ((base_length/2) - x_offset)} ${y_reflect * base_width/2} ${-z_offset}" rpy= "0 0 0"/>
-            <axis xyz = "0 1 0"/>
-        </joint>
-        <link name="${prefix}_wheel_link">
-            <collision>
-                <origin xyz="0 ${wheel_length/2} 0" rpy= "${pi/2} 0 0"/>
-                <geometry>
-                    <cylinder radius="${wheel_radius}" length="${wheel_length}"/>
-                </geometry>
-            </collision>
-            <visual>
-                <origin xyz="0 ${y_reflect * wheel_length/2} 0" rpy="${pi/2} 0 0"/>
-                <geometry>
-                    <cylinder radius="${wheel_radius}" length="${wheel_length}"/>
-                </geometry>
-                <material name="black"/>
-            </visual>
-            <xacro:cylinder_inertia m="${wheel_mass}" r="${wheel_radius}" h="${wheel_length}"/>
-        </link>
-    </xacro:macro>
-    <!-- call macros to define wheels-->
-    <xacro:wheel prefix="front_left" x_reflect="1" y_reflect="1"/>
-    <xacro:wheel prefix="front_right" x_reflect="1" y_reflect="-1"/>
-    <xacro:wheel prefix="back_left" x_reflect="-1" y_reflect="1"/>
-    <xacro:wheel prefix="back_right" x_reflect="-1" y_reflect="-1"/>
+  <!-- Virtual frame: no mass, inertia, or geometry. -->
+  <link
+    name="base_footprint" />
+  <joint
+    name="base_footprint_joint"
+    type="fixed">
+    <!-- base_footprint lies on the ground plane under base_link (150 mm
+         effective wheel radius; the grousers sink into the terrain). -->
+    <origin
+      xyz="0 0 0.264385282852235"
+      rpy="0 0 0" />
+    <parent
+      link="base_footprint" />
+    <child
+      link="base_link" />
+    <axis
+      xyz="0 0 0" />
+  </joint>
+  <link
+    name="base_link">
+    <inertial>
+      <origin
+        xyz="-0.0054525 0.0030219 -0.021701"
+        rpy="0 0 0" />
+      <mass
+        value="7.6408" />
+      <inertia
+        ixx="0.027157"
+        ixy="1.7861E-05"
+        ixz="2.7978E-05"
+        iyy="0.085655"
+        iyz="2.5148E-06"
+        izz="0.10185" />
+    </inertial>
+    <visual>
+      <!-- SolidWorks exported base_link.STL relative to a frame 0.264385 m
+           below base_link, so shift it back up into base_link. -->
+      <origin
+        xyz="0 0 -0.264385282852235"
+        rpy="0 0 0" />
+      <geometry>
+        <mesh
+          filename="package://rosey_description/description/meshes/base_link.STL" />
+      </geometry>
+      <material
+        name="base_link_material">
+        <color
+          rgba="0.75294 0.75294 0.75294 1" />
+      </material>
+    </visual>
+    <collision>
+      <!-- SolidWorks exported base_link.STL relative to a frame 0.264385 m
+           below base_link, so shift it back up into base_link. -->
+      <origin
+        xyz="0 0 -0.264385282852235"
+        rpy="0 0 0" />
+      <geometry>
+        <mesh
+          filename="package://rosey_description/description/meshes/base_link.STL" />
+      </geometry>
+    </collision>
+  </link>
+  <!-- Virtual frame: no mass, inertia, or geometry. -->
+  <link
+    name="imu_link" />
+  <joint
+    name="imu_joint"
+    type="fixed">
+    <origin
+      xyz="0.16256 -0.05 0.017088"
+      rpy="0 0 0" />
+    <parent
+      link="base_link" />
+    <child
+      link="imu_link" />
+    <axis
+      xyz="0 0 0" />
+  </joint>
+  <link
+    name="front_left_wheel_link">
+    <inertial>
+      <origin
+        xyz="-9.6438E-08 -0.0035297 2.5028E-08"
+        rpy="0 0 0" />
+      <mass
+        value="0.8653" />
+      <inertia
+        ixx="0.0018675"
+        ixy="1.302E-10"
+        ixz="-1.4777E-08"
+        iyy="0.00325"
+        iyz="-1.3427E-10"
+        izz="0.0018676" />
+    </inertial>
+    <visual>
+      <origin
+        xyz="0 0 0"
+        rpy="0 0 0" />
+      <geometry>
+        <mesh
+          filename="package://rosey_description/description/meshes/front_left_wheel_link.STL" />
+      </geometry>
+      <material
+        name="front_left_wheel_link_material">
+        <color
+          rgba="0.75294 0.75294 0.75294 1" />
+      </material>
+    </visual>
+    <collision>
+      <origin
+        xyz="0 0 0"
+        rpy="0 0 0" />
+      <geometry>
+        <mesh
+          filename="package://rosey_description/description/meshes/front_left_wheel_link.STL" />
+      </geometry>
+    </collision>
+  </link>
+  <joint
+    name="front_left_wheel_joint"
+    type="continuous">
+    <origin
+      xyz="0.1881 0.16825 -0.11444"
+      rpy="0 0 0" />
+    <parent
+      link="base_link" />
+    <child
+      link="front_left_wheel_link" />
+    <axis
+      xyz="0 1 0" />
+  </joint>
+  <link
+    name="front_right_wheel_link">
+    <inertial>
+      <origin
+        xyz="9.6438E-08 0.0035297 2.5028E-08"
+        rpy="0 0 0" />
+      <mass
+        value="0.8653" />
+      <inertia
+        ixx="0.0018675"
+        ixy="1.302E-10"
+        ixz="1.4777E-08"
+        iyy="0.00325"
+        iyz="1.3427E-10"
+        izz="0.0018676" />
+    </inertial>
+    <visual>
+      <origin
+        xyz="0 0 0"
+        rpy="0 0 0" />
+      <geometry>
+        <mesh
+          filename="package://rosey_description/description/meshes/front_right_wheel_link.STL" />
+      </geometry>
+      <material
+        name="front_right_wheel_link_material">
+        <color
+          rgba="0.75294 0.75294 0.75294 1" />
+      </material>
+    </visual>
+    <collision>
+      <origin
+        xyz="0 0 0"
+        rpy="0 0 0" />
+      <geometry>
+        <mesh
+          filename="package://rosey_description/description/meshes/front_right_wheel_link.STL" />
+      </geometry>
+    </collision>
+  </link>
+  <joint
+    name="front_right_wheel_joint"
+    type="continuous">
+    <origin
+      xyz="0.1881 -0.16825 -0.11433"
+      rpy="0 0 0" />
+    <parent
+      link="base_link" />
+    <child
+      link="front_right_wheel_link" />
+    <axis
+      xyz="0 1 0" />
+  </joint>
+  <link
+    name="back_left_wheel_link">
+    <inertial>
+      <origin
+        xyz="-9.6438E-08 -0.0035297 2.5028E-08"
+        rpy="0 0 0" />
+      <mass
+        value="0.8653" />
+      <inertia
+        ixx="0.0018675"
+        ixy="1.302E-10"
+        ixz="-1.4777E-08"
+        iyy="0.00325"
+        iyz="-1.3427E-10"
+        izz="0.0018676" />
+    </inertial>
+    <visual>
+      <origin
+        xyz="0 0 0"
+        rpy="0 0 0" />
+      <geometry>
+        <mesh
+          filename="package://rosey_description/description/meshes/back_left_wheel_link.STL" />
+      </geometry>
+      <material
+        name="back_left_wheel_link_material">
+        <color
+          rgba="0.75294 0.75294 0.75294 1" />
+      </material>
+    </visual>
+    <collision>
+      <origin
+        xyz="0 0 0"
+        rpy="0 0 0" />
+      <geometry>
+        <mesh
+          filename="package://rosey_description/description/meshes/back_left_wheel_link.STL" />
+      </geometry>
+    </collision>
+  </link>
+  <joint
+    name="back_left_wheel_joint"
+    type="continuous">
+    <origin
+      xyz="-0.1881 0.16825 -0.11433"
+      rpy="0 0 0" />
+    <parent
+      link="base_link" />
+    <child
+      link="back_left_wheel_link" />
+    <axis
+      xyz="0 1 0" />
+  </joint>
+  <link
+    name="back_right_wheel_link">
+    <inertial>
+      <origin
+        xyz="9.6438E-08 0.0035297 2.5028E-08"
+        rpy="0 0 0" />
+      <mass
+        value="0.8653" />
+      <inertia
+        ixx="0.0018675"
+        ixy="1.302E-10"
+        ixz="1.4777E-08"
+        iyy="0.00325"
+        iyz="1.3427E-10"
+        izz="0.0018676" />
+    </inertial>
+    <visual>
+      <origin
+        xyz="0 0 0"
+        rpy="0 0 0" />
+      <geometry>
+        <mesh
+          filename="package://rosey_description/description/meshes/back_right_wheel_link.STL" />
+      </geometry>
+      <material
+        name="back_right_wheel_link_material">
+        <color
+          rgba="0.75294 0.75294 0.75294 1" />
+      </material>
+    </visual>
+    <collision>
+      <origin
+        xyz="0 0 0"
+        rpy="0 0 0" />
+      <geometry>
+        <mesh
+          filename="package://rosey_description/description/meshes/back_right_wheel_link.STL" />
+      </geometry>
+    </collision>
+  </link>
+  <joint
+    name="back_right_wheel_joint"
+    type="continuous">
+    <origin
+      xyz="-0.1881 -0.16825 -0.11444"
+      rpy="0 0 0" />
+    <parent
+      link="base_link" />
+    <child
+      link="back_right_wheel_link" />
+    <axis
+      xyz="0 1 0" />
+  </joint>
+  <link
+    name="camera_0_link">
+    <inertial>
+      <origin
+        xyz="-0.0046466 0.00022408 0.0091953"
+        rpy="0 0 0" />
+      <mass
+        value="0.019933" />
+      <inertia
+        ixx="1.1262E-05"
+        ixy="-4.5237E-08"
+        ixz="9.1405E-07"
+        iyy="6.1143E-06"
+        iyz="8.1423E-08"
+        izz="7.1098E-06" />
+    </inertial>
+    <visual>
+      <origin
+        xyz="0 0 0"
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
File: src/rosey_description/description/ros2_control/roseybot_control.urdf.xacro (robot description, xacro)
@@ -4,4 +4,6 @@
         <joint name="${prefix}_wheel_joint">
             <command_interface name="velocity"/>
+            <!-- RoseyBotSystemHardware expects exactly these five state
+                 interfaces, with position first and velocity second. -->
             <state_interface name="position"/>
             <state_interface name="velocity"/>
@@ -11,24 +13,31 @@
         </joint>
     </xacro:macro>
-    <ros2_control name="roseybot_teensy" type="system">
-        <hardware>
-          <plugin>roseybot_arduino/RoseyBotSystemHardware</plugin>
-          <param name="baud">115200</param>
-          <param name="timeout_ms">150</param>
-          <param name="device">/dev/ttyACM0</param>
-          <param name="enc/rev">5281.1</param>
-          <!-- safety_check tuning parameters -->
-          <param name="noise_floor_percent">2</param>
-          <param name="opposite_direction_ms">500</param>
-          <param name="max_velocity_percent">75</param>
-        </hardware>
-        <!-- <hardware>
-          <plugin>mock_components/GenericSystem</plugin>
-          <param name="calculate_dynamics">true</param>
-        </hardware> -->
-        <xacro:connect_joint prefix="front_left"/>
-        <xacro:connect_joint prefix="front_right"/>
-        <xacro:connect_joint prefix="back_left"/>
-        <xacro:connect_joint prefix="back_right"/>
-    </ros2_control>
+    <xacro:macro name="roseybot_ros2_control" params="use_mock_hardware">
+        <ros2_control name="roseybot_teensy" type="system">
+            <hardware>
+                <xacro:if value="${use_mock_hardware}">
+                    <plugin>mock_components/GenericSystem</plugin>
+                    <param name="calculate_dynamics">true</param>
+                </xacro:if>
+                <xacro:unless value="${use_mock_hardware}">
+                    <plugin>roseybot_arduino/RoseyBotSystemHardware</plugin>
+                    <param name="baud">115200</param>
+                    <param name="timeout_ms">150</param>
+                    <param name="device">/dev/ttyACM0</param>
+                    <param name="enc/rev">5281.1</param>
+                    <!-- safety_check tuning parameters -->
+                    <param name="noise_floor_percent">2</param>
+                    <param name="opposite_direction_ms">500</param>
+                    <param name="max_velocity_percent">75</param>
+                </xacro:unless>
+            </hardware>
+            <!-- Do not reorder: RoseyBotSystemHardware maps joints by index.
+                 Telemetry index i is motor i+1 (FL, FR, BL, BR), and write()
+                 sends joint 0 as the left command and joint 1 as the right. -->
+            <xacro:connect_joint prefix="front_left"/>
+            <xacro:connect_joint prefix="front_right"/>
+            <xacro:connect_joint prefix="back_left"/>
+            <xacro:connect_joint prefix="back_right"/>
+        </ros2_control>
+    </xacro:macro>
 </robot>

File: src/rosey_description/description/urdf/roseybot.urdf.xacro (robot description, xacro)
@@ -3,8 +3,7 @@
 <robot xmlns:xacro="http://www.ros.org/wiki/xacro" name="roseybot">
   <xacro:arg name="use_mock_hardware" default="false" />
-  <!-- Import Rviz colors -->
-  <xacro:include filename="$(find rosey_description)/description/robot/roseybot_colors.urdf.xacro" />
   <xacro:include filename="$(find rosey_description)/description/robot/roseybot_description.urdf.xacro"/>
   <!-- Import ros2_control hardware description -->
   <xacro:include filename="$(find rosey_description)/description/ros2_control/roseybot_control.urdf.xacro" />
+  <xacro:roseybot_ros2_control use_mock_hardware="$(arg use_mock_hardware)"/>
 </robot>

Commit message: fixed realsense joint / link

File: src/rosey_description/description/robot/roseybot_description.urdf.xacro (robot description, xacro)
@@ -632,5 +632,5 @@
     <inertial>
       <origin
-        xyz="0.0122023502976824 -0.0474592338080081 -0.0126678739124035"
+        xyz="-0.0091476 -0.047459 -0.012668"
         rpy="0 0 0" />
       <mass
@@ -645,6 +645,7 @@
     </inertial>
     <visual>
-      <origin
-        xyz="0 0 0"
+      <!-- offset compensates for realsense_link origin moved +21.347 mm along link x; STL is referenced to the old origin -->
+      <origin
+        xyz="-0.021347 0 0"
         rpy="0 0 0" />
       <geometry>
@@ -660,5 +661,5 @@
     <collision>
       <origin
-        xyz="0 0 0"
+        xyz="-0.021347 0 0"
         rpy="0 0 0" />
       <geometry>
@@ -672,5 +673,5 @@
     type="fixed">
     <origin
-      xyz="0.21558 0.04725 0.22826"
+      xyz="0.236602527122989 0.0472499999999953 0.224551697487006"
       rpy="0 0.17453 0" />
     <parent
